File: PCB/mote backpack/mote backpack.kicad_pcb (KiCad board)
At the start: 2 copper layers, 62 x 37 mm, 15 parts, among them J1 DF17_2.0_-30DP-0.5V_57_, J2 73251-1350, J3 Micro_SD_Card_Det2, J4 Conn_01x06_Socket, U1 MAX3232, U3 ADAFRUIT_QT_PY

Commit message: test that changes tracked
Parts:
- added J5: D45V5F12, Connector_PinHeader_2.54mm:PinHeader_1x03_P2.54mm_Vertical, F.Cu at (176.8, 108.7)
